File: Killswitch Module.kicad_sch (KiCad schematic)
At the start: 0 parts

Commit message: push changes i forgot what they were
Changed lines of the file:
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@@
 	(generator_version "10.0")
 	(paper "A4")
+	(hierarchical_label "GND"
+		(shape input)
+		(at 5.3848 5.8896 0)
+		(effects
+			(font
+				(size 1.27 1.27)
+			)
+			(justify left)
+		)
+	)
 	(hierarchical_label "14V8 IN"
 		(shape input)
@@
 		(effects
 			(font
+				(size 1.27 1.27)
+			)
+			(justify right)
+		)
+	)
+	(hierarchical_label "GND"
+		(shape passive)
+		(at 3.3496 7.9474 90)
+		(effects
+			(font
+				(size 1.27 1.27)
+			)
+			(justify left)
+		)
+	)
+	(hierarchical_label "KILL1"
+		(shape input)
+		(at 8.4296 7.9248 270)
+		(effects
+			(font
